File: mcu.sch (KiCad schematic (older format))
At the start: 35 parts, among them J4 UEXT, J7 6P6C, J8 ST_Nucleo_SWD_5p, U1 STM32L072CZTx, U4 D1213A-04SO

Commit message: Updates after manufacturer feedback
Parts:
- J4: Manufacturer any -> On Shore Technology Inc.; PartNumber (none) -> 302-S101
- LED1, LED2, LED3, LED5: footprint LED_THT:LED_D3.0mm -> LibreSolar:LED_0603_D3.0mm
Connections:
- net RX: now reaches J7.2, R43.1, U4.6
- net TX: now reaches J7.3, R44.1, U4.4
Changed lines of the file:
@@
 EESchema Schematic File Version 4
 LIBS:pwm_charger_20a-cache
-EELAYER 26 0
+EELAYER 29 0
 EELAYER END
 $Descr A4 11693 8268
@@
 Sheet 3 4
 Title "PWM Solar Charge Controller"
-Date "2019-03-05"
-Rev "0.2"
+Date "2019-04-25"
+Rev "0.2.1"
 Comp "Libre Solar"
 Comment1 "Author: Martin Jäger"
@@
 F 0 "LED4" H 5225 6550 50  0000 L CNN
 F 1 "green" H 5225 6450 50  0000 L CNN
-F 2 "LED_THT:LED_D3.0mm" V 5100 6500 50  0001 C CNN
+F 2 "LibreSolar:LED_0603_D3.0mm" V 5100 6500 50  0001 C CNN
 F 3 "" V 5100 6500 50  0000 C CNN
 F 4 "Lite-On" H 0   0   50  0001 C CNN "Manufacturer"
@@
 F 2 "LibreSolar:Box_Header_2x05x2.54mm_Straight" H 7800 1200 50  0001 C CIN
 F 3 "" H 7800 1800 60  0000 C CNN
-F 4 "any" H 0   0   50  0001 C CNN "Manufacturer"
-F 5 "2x5 pin box header, pitch 2.54 mm" H 0   0   50  0001 C CNN "Remarks"
+F 4 "On Shore Technology Inc." H 0   0   50  0001 C CNN "Manufacturer"
+F 5 "302-S101" H 7800 1800 50  0001 C CNN "PartNumber"
+F 6 "2x5 pin box header, pitch 2.54 mm" H 0   0   50  0001 C CNN "Remarks"
 	1    7800 1800
 	1    0    0    -1
@@
 F 0 "LED5" H 5725 6550 50  0000 L CNN
 F 1 "green" H 5725 6450 50  0000 L CNN
-F 2 "LED_THT:LED_D3.0mm" V 5600 6500 50  0001 C CNN
+F 2 "LibreSolar:LED_0603_D3.0mm" V 5600 6500 50  0001 C CNN
 F 3 "" V 5600 6500 50  0000 C CNN
 F 4 "Lite-On" H 0   0   50  0001 C CNN "Manufacturer"
@@
 F 0 "LED1" H 5225 5950 50  0000 L CNN
 F 1 "yellow" H 5225 5850 50  0000 L CNN
-F 2 "LED_THT:LED_D3.0mm" V 5100 5900 50  0001 C CNN
+F 2 "LibreSolar:LED_0603_D3.0mm" V 5100 5900 50  0001 C CNN
 F 3 "" V 5100 5900 50  0000 C CNN
 F 4 "Lite-On" H 0   0   50  0001 C CNN "Manufacturer"
@@
 F 0 "LED3" H 6225 5950 50  0000 L CNN
 F 1 "yellow" H 6225 5850 50  0000 L CNN
-F 2 "LED_THT:LED_D3.0mm" V 6100 5900 50  0001 C CNN
+F 2 "LibreSolar:LED_0603_D3.0mm" V 6100 5900 50  0001 C CNN
 F 3 "" V 6100 5900 50  0000 C CNN
 F 4 "Lite-On" H 0   0   50  0001 C CNN "Manufacturer"
@@
 F 0 "LED2" H 5725 5950 50  0000 L CNN
 F 1 "yellow" H 5725 5850 50  0000 L CNN
-F 2 "LED_THT:LED_D3.0mm" V 5600 5900 50  0001 C CNN
+F 2 "LibreSolar:LED_0603_D3.0mm" V 5600 5900 50  0001 C CNN
 F 3 "" V 5600 5900 50  0000 C CNN
 F 4 "Lite-On" H 0   0   50  0001 C CNN "Manufacturer"
@@
 Wire Wire Line
 	8600 2900 8600 3000
+Text Label 7000 3700 0    50   ~ 0
+RX
+Text Label 7000 3800 0    50   ~ 0
+TX
 $EndSCHEMATC
