File: power_supply.sch (KiCad schematic (older format))
At the start: 25 parts, among them J5 USB_A, T5 MMBT3904, U3 MC34063AD, U5 LP2950-3.3_TO252

Commit message: Updates after manufacturer feedback
Parts:
- D2, D9: footprint Diode_SMD:D_SOD-123F -> LibreSolar:D_SOD-123F
Changed lines of the file:
@@
 EESchema Schematic File Version 4
 LIBS:pwm_charger_20a-cache
-EELAYER 26 0
+EELAYER 29 0
 EELAYER END
 $Descr A4 11693 8268
@@
 Sheet 4 4
 Title "PWM Solar Charge Controller"
-Date "2019-03-05"
-Rev "0.2"
+Date "2019-04-25"
+Rev "0.2.1"
 Comp "Libre Solar"
 Comment1 "Author: Martin Jäger"
@@
 F 0 "D9" V 6754 2879 50  0000 L CNN
 F 1 "SS14FL" V 6845 2879 50  0000 L CNN
-F 2 "Diode_SMD:D_SOD-123F" V 6800 2800 50  0001 C CNN
+F 2 "LibreSolar:D_SOD-123F" V 6800 2800 50  0001 C CNN
 F 3 "" V 6800 2800 50  0000 C CNN
 F 4 "On Semiconductor" H 0   0   50  0001 C CNN "Manufacturer"
@@
 F 0 "D2" V 1654 2079 50  0000 L CNN
 F 1 "SS14FL" V 1745 2079 50  0000 L CNN
-F 2 "Diode_SMD:D_SOD-123F" V 1700 2000 50  0001 C CNN
+F 2 "LibreSolar:D_SOD-123F" V 1700 2000 50  0001 C CNN
 F 3 "" V 1700 2000 50  0000 C CNN
 F 4 "On Semiconductor" H 0   0   50  0001 C CNN "Manufacturer"
