File: kicad/power_supply.sch (KiCad schematic (older format))
At the start: 25 parts, among them J5 USB_A, T5 MMBT3904, U3 MC34063AD, U5 LP2950-3.3_TO252

Commit message: Improved power supply and exposed BOOT0 pin
- BOOT0 pin connected to BUTTON wire to allow firmware upgrade via LS.one port
- Additional emitter follower for 3V3 power supply to increase margin to 30V absolute max. rating of LDO in case of 24V battery
- Corners adjusted to match shape of MPPT 1210 HUS
Parts:
- added D3: 12V, Diode_SMD:D_SOT-23_ANK, symbol Project:D_Zener
- added R35: 12k, LibreSolar:R_0805_2012, symbol Project:R
- added T6: MMBT3904, LibreSolar:SOT-23, symbol Transistor_BJT:MMBT3904
- T5: symbol Transistor_BJT:BC817 -> Transistor_BJT:MMBT3904
Connections:
- net +12V: now also D3.2 (A)
- net BAT_INPUT: now reaches C13.1, C6.1, D2.1 (K), R31.2, R36.2, T5.3 (C), U3.6 (Vin)
- net BAT_INPUT: now also R35.2, T6.3 (C); no longer C14.1, U5.1 (VI)
- new net: C14.1, T6.2 (E), U5.1 (VI)
- new net: D3.1 (K), R35.1, T6.1 (B)
Other:
- note added: "Drop part of the voltage\nin 24V systems to stay below\n30V absolute max of LP2950"
- moved on the sheet: C14, C15, C22, D8, R31, T5, TP8, TP9, U5
